Commit message: add support for training controller for 4+2 config using PPO

File: resources/robots/hexa/hexa2.urdf (robot description, URDF)
Before this commit: robot hexarotor, 13 links, 12 joints
Links:
- added link wing, mass 0.005; collision box size=0.4 0.08 0.005; visual box size=0.4 0.08 0.005
Joints:
- added joint base_to_wing: type fixed, parent base_link, child wing, origin xyz=0 0 0 rpy=0 0 1.5708
